Commit message: working on chassis; rviz first config

File: arm_urdf/urdf/chassis.xacro (robot description, xacro)
@@ -1,6 +1,61 @@
 <?xml version="1.0" ?>
 <robot name="robot" xmlns:xacro="http://www.ros.org/wiki/xacro">
+<!-- chassis and front caster wheel -->
 <link name="base_link">
-	<!-- ... -->
+	<pose>0 0 0.1 0 0 0</pose>
+	<inertial>
+		<mass
+			value="5" />
+		<origin
+			rpy="0 0 0"
+			xyz="0 0 0.1"/>
+		<inertia
+			ixx="0.0395416666667" iyy="0.106208333333" izz="0.106208333333"
+			ixy="0" ixz="0" iyz="0" />
+	</inertial>
+    <!-- collision and visual chassis -->
+	<collision name="collision_chassis">
+		<geometry>
+			<box size="0.5 0.3 0.07"/>
+		</geometry>
+	</collision>
+    <visual>
+		<origin rpy="0 0 0" xyz="0 0 0"/>
+		<geometry>
+			<box size="0.5 0.3 0.07"/>
+		</geometry>
+		<material name="blue"/>
+	</visual>
+	<!-- collision and visual chassis -->
+    <!-- collision, physics and visual of the front caster wheel -->
+	<collision name="caster_front_collision">
+		<origin
+			rpy=" 0 0 0"
+			xyz="0.35 0 -0.05"/>
+		<geometry>
+			<sphere radius="0.05"/>
+		</geometry>
+		<surface>
+			<friction>
+				<ode>
+					<mu>0</mu>
+					<mu2>0</mu2>
+					<slip1>1.0</slip1>
+					<slip2>1.0</slip2>
+				</ode>
+			</friction>
+		</surface>
+	</collision>
+	<visual name="caster_front_visual">
+		<origin
+			rpy=" 0 0 0"
+			xyz="0.2 0 -0.05"/>
+		<geometry>
+			<sphere radius="0.05"/>
+		</geometry>
+	</visual>
+	<!-- collision, physics and visual of the front caster wheel -->
 </link>
+<!-- chassis and front caster wheel -->
+<!--  -->
 </robot>

File: arm_urdf/urdf/main.xacro (robot description, xacro)
@@ -4,5 +4,5 @@
 <xacro:include filename="macros.xacro"/>
 <xacro:include filename="params.xacro"/>
-<!-- <xacro:include filename="materials.xacro"/> -->
+<xacro:include filename="materials.xacro"/>
 <!-- <xacro:include filename="gazebo.gazebo"/> -->
 <!-- <xacro:include filename="transmission.xacro"/> -->

Commit message: VISUALIZATION ISSUE with RViz SOLVED

File: arm_urdf/urdf/chassis.xacro (robot description, xacro)
@@ -58,4 +58,11 @@
 </link>
 <!-- chassis and front caster wheel -->
-<!--  -->
+<!-- Wheels -->
+<xacro:link_wheel name="link_right_wheel" />
+<xacro:joint_wheel name="joint_right_wheel"
+	child="link_right_wheel" parent="base_link" xx="-0.05" yy="0.15" zz="0"  />
+<xacro:link_wheel name="link_left_wheel" />
+<xacro:joint_wheel name="joint_left_wheel"
+	child="link_left_wheel" parent="base_link" xx="-0.05" yy="-0.15" zz="0"  />
+<!-- Wheels -->
 </robot>

File: arm_urdf/urdf/macros.xacro (robot description, xacro)
@@ -14,4 +14,7 @@
 <xacro:macro name="link_wheel" params="name">
 	<link name="${name}">
+		<origin
+			xyz="0 0 0"
+			rpy="0 0 0"/>
 		<inertial>
 			<mass value="0.2"/>
@@ -42,11 +45,11 @@
 </xacro:macro>
 <!-- joint of the wheel on the chassis -->
-<xacro:macro name="joint_wheel" params="name child origin_xyz">
+<xacro:macro name="joint_wheel" params="name child parent xx yy zz">
 	<joint name="${name}" type="continuous">
-		<parent link="base_link"/>
+		<parent link="${parent}"/>
 		<child link="${child}"/>
 		<origin
 			rpy="0 0 0"
-			xyz="${origin_xyz}"/>
+			xyz="${xx} ${yy} ${zz}"/>
         <axis
 			rpy="0 0 0"

File: arm_urdf/urdf/main.xacro (robot description, xacro)
@@ -15,4 +15,5 @@
 </link>
 <!-- robot chassis -->
+<xacro:include filename="chassis.xacro"></xacro:include>
 <joint name="root_joint" type="fixed">
 	<parent link="root_link"/>
@@ -20,6 +21,6 @@
 	<origin xyz="0 0 0" rpy="0 0 0"/>
 </joint>
-<xacro:include filename="chassis.xacro"></xacro:include>
 <!-- robot manipulator -->
+<xacro:include filename="arm.xacro"></xacro:include>
 <joint name="arm_base_to_base" type="fixed">
 	<parent link="base_link"/>
@@ -27,4 +28,3 @@
 	<origin xyz="0 0 0" rpy="0 0 0"/>
 </joint>
-<xacro:include filename="arm.xacro"></xacro:include>
 </robot>

File: arm_urdf/urdf/model.urdf (robot description, URDF)
Before this commit: robot robot, 3 links, 2 joints
Links:
- added link link_left_wheel, mass 0.2; collision cylinder length=0.04 radius=0.1; visual cylinder length=0.04 radius=0.1
- added link link_right_wheel, mass 0.2; collision cylinder length=0.04 radius=0.1; visual cylinder length=0.04 radius=0.1
- link base_link: mass None -> 5; geometry collision box size=0.5 0.3 0.07; collision sphere radius=0.05
Joints:
- added joint joint_left_wheel: type continuous, parent base_link, child link_left_wheel, origin xyz=-0.05 -0.15 0 rpy=0 0 0, axis 0 1 0, limit effort=10000 velocity=1000
- added joint joint_right_wheel: type continuous, parent base_link, child link_right_wheel, origin xyz=-0.05 0.15 0 rpy=0 0 0, axis 0 1 0, limit effort=10000 velocity=1000

Commit message: chassis implementation

File: arm_urdf/urdf/chassis.xacro (robot description, xacro)
@@ -58,4 +58,31 @@
 </link>
 <!-- chassis and front caster wheel -->
+<!-- place for laser sensors -->
+<link name="laser">
+	<inertial>
+		<origin xyz="0 0 0" rpy="0 0 0" />
+		<mass value="1" />
+		<xacro:cylinder_inertia mass="1" r="0.05" l="0.1" />
+	</inertial>
+	<visual>
+		<origin xyz="0 0 0" rpy="0 0 0" />
+		<geometry>
+			<cylinder radius="0.05" length="0.1"/>
+		</geometry>
+		<material name="white" />
+	</visual>
+	<collision>
+		<origin xyz="0 0 0" rpy="0 0 0"/>
+		<geometry>
+			<cylinder radius="0.05" length="0.1"/>
+		</geometry>
+	</collision>
+</link>
+<joint name="joint_laser" type="fixed">
+	<parent link="base_link"/>
+	<child link="laser"/>
+	<origin xyz="0.15 0 0.05" rpy="0 0 0"/>
+</joint>
+<!-- place for laser sensors -->
 <!-- Wheels -->
 <xacro:link_wheel name="link_right_wheel" />
