Commit message: minor changes; deleted not working moveit pkg

File: arm_urdf/urdf/main.xacro (robot description, xacro)
@@ -6,5 +6,4 @@
 <xacro:include filename="materials.xacro"/>
 <xacro:include filename="gazebo.gazebo"/>
-<xacro:include filename="transmission.xacro"/>
 <!-- dummy link (model root) -->
 <!-- see this post :
@@ -29,3 +28,4 @@
 	<origin xyz="0 0 0.085" rpy="0 0 0"/>
 </joint>
+<xacro:include filename="transmission.xacro"/>
 </robot>

File: arm_urdf/urdf/model.urdf (robot description, URDF)
Before this commit: robot robot, 5 links, 4 joints
Links:
- added link arm_link_01, mass 0.025; collision cylinder length=0.2 radius=0.04; visual cylinder length=0.2 radius=0.04
- added link arm_link_02, mass 0.025; collision cylinder length=0.2 radius=0.04; visual cylinder length=0.2 radius=0.04
- added link arm_link_03, mass 0.025; collision cylinder length=0.2 radius=0.04; visual cylinder length=0.2 radius=0.04
- added link arm_link_04, mass 0.025; collision box size=0.034 0.2 0.08; visual box size=0.034 0.2 0.08
- added link laser, mass 1; collision cylinder length=0.1 radius=0.05; visual cylinder length=0.1 radius=0.05
- added link left_grip_link, mass 0.01; collision box size=0.06 0.02 0.08; visual box size=0.06 0.02 0.08
- added link right_grip_link, mass 0.01; collision box size=0.06 0.02 0.08; visual box size=0.06 0.02 0.08
- link arm_base_link: mass None -> 0.1; geometry collision box size=0.1 0.1 0.1; visual box size=0.1 0.1 0.1
Joints:
- added joint arm_joint_01: type revolute, parent arm_base_link, child arm_link_01, origin xyz=0 0 0.05 rpy=0 0 0, axis 0 0 1, limit lower=-3.12 upper=3.139 effort=1000.0 velocity=5
- added joint arm_joint_02: type revolute, parent arm_link_01, child arm_link_02, origin xyz=0 0 0.2 rpy=0 0 0, axis 0 1 0, limit lower=-1.8 upper=1.8 effort=1000.0 velocity=5
- added joint arm_joint_03: type revolute, parent arm_link_02, child arm_link_03, origin xyz=0 0 0.2 rpy=0 0 0, axis 0 1 0, limit lower=-1.8 upper=1.8 effort=1000.0 velocity=5
- added joint arm_joint_04: type revolute, parent arm_link_03, child arm_link_04, origin xyz=0 0 0.2 rpy=0 0 0, axis 0 1 0, limit lower=-1.8 upper=1.8 effort=10000.0 velocity=5
- added joint joint_laser: type fixed, parent base_link, child laser, origin xyz=0.15 0 0.05 rpy=0 0 0
- added joint left_grip_joint: type prismatic, parent arm_link_04, child left_grip_link, origin xyz=0.045 -0.05 0.04 rpy=0 0 0, axis 0 1 0, limit lower=-0.035 upper=0.04 effort=1000.0 velocity=6.5
- added joint right_grip_joint: type prismatic, parent arm_link_04, child right_grip_link, origin xyz=0.045 0.05 0.04 rpy=0 0 0, axis 0 1 0, limit lower=-0.04 upper=0.035 effort=1000.0 velocity=6.5
- joint arm_base_to_base: origin xyz=0 0 0 rpy=0 0 0 -> xyz=0 0 0.085 rpy=0 0 0

Commit message: ISSUE unable to load controllers (seems) SOLVED

File: arm_urdf/urdf/main.xacro (robot description, xacro)
@@ -22,7 +22,9 @@
 <!-- robot manipulator -->
 <xacro:include filename="arm.xacro"></xacro:include>
-<joint name="arm_base_to_base" type="fixed">
+<joint name="arm_base_to_base" type="revolute">
 	<parent link="base_link"/>
 	<child  link="arm_base_link"/>
+	<axis xyz="0 0 1" />
+	<limit effort="1000.0" lower="-1.8" upper="1.8" velocity="5"/>
 	<!-- origin : 0.5*(chassis height) + 0.5*(arm base link height) -->
 	<origin xyz="0 0 0.085" rpy="0 0 0"/>

File: arm_urdf/urdf/model/model.urdf (robot description, URDF)
Before this commit: robot robot, 12 links, 11 joints
Joints:
- joint arm_base_to_base: axis (none) -> 0 0 1; limit (none) -> lower=-1.8 upper=1.8 effort=1000.0 velocity=5; type fixed -> revolute

File: arm_urdf/urdf/transmission.xacro (robot description, xacro)
@@ -1,4 +1,37 @@
 <?xml version="1.0" ?>
 <robot name="m2wr" xmlns:xacro="https://www.ros.org/wiki/xacro" >
+<!-- CHASSIS HARDWARE INTERFACE -->
+<transmission name="trans_joint_right_wheel">
+	<type>transmission_interface/SimpleTransmission</type>
+	<joint name="joint_right_wheel">
+		<hardwareInterface>hardware_interface/EffortJointInterface</hardwareInterface>
+	</joint>
+	<actuator name="joint_right_wheel_motor">
+		<hardwareInterface>hardware_interface/EffortJointInterface</hardwareInterface>
+		<mechanicalReduction>1</mechanicalReduction>
+	</actuator>
+</transmission>
+<transmission name="trans_joint_left_wheel">
+	<type>transmission_interface/SimpleTransmission</type>
+	<joint name="joint_left_wheel">
+            <hardwareInterface>hardware_interface/EffortJointInterface</hardwareInterface>
+	</joint>
+	<actuator name="joint_left_wheel_motor">
+		<hardwareInterface>hardware_interface/EffortJointInterface</hardwareInterface>
+		<mechanicalReduction>1</mechanicalReduction>
+	</actuator>
+</transmission>
+<!-- CHASSIS HARDWARE INTERFACE -->
+<!-- ARM TRANSMISSION -->
+<transmission name="trans_arm_base_to_base">
+	<type>transmission_interface/SimpleTransmission</type>
+	<joint name="arm_base_to_base">
+		<hardwareInterface>hardware_interface/EffortJointInterface</hardwareInterface>
+	</joint>
+	<actuator name="arm_base_to_base_motor">
+		<hardwareInterface>hardware_interface/EffortJointInterface</hardwareInterface>
+		<mechanicalReduction>1</mechanicalReduction>
+	</actuator>
+</transmission>
 <transmission name="arm_joint_01_trans">
 	<type>transmission_interface/SimpleTransmission</type>
@@ -61,3 +94,4 @@
 	</actuator>
 </transmission>
+<!-- ARM TRANSMISSION -->
 </robot>
