Commit message: first test of the model, ready to write more; updated readme

File: arm_urdf/urdf/arm.xacro (robot description, xacro)
@@ -1,3 +1,6 @@
 <?xml version="1.0" ?>
 <robot name="robot" xmlns:xacro="http://www.ros.org/wiki/xacro">
+<link name="arm_base_link">
+	<!-- ... -->
+</link>
 </robot>

File: arm_urdf/urdf/chassis.xacro (robot description, xacro)
@@ -1,3 +1,6 @@
 <?xml version="1.0" ?>
 <robot name="robot" xmlns:xacro="http://www.ros.org/wiki/xacro">
+<link name="base_link">
+	<!-- ... -->
+</link>
 </robot>

File: arm_urdf/urdf/main.xacro (robot description, xacro)
@@ -4,8 +4,11 @@
 <xacro:include filename="macros.xacro"/>
 <xacro:include filename="params.xacro"/>
-<xacro:include filename="materials.xacro"/>
-<xacro:include filename="gazebo.gazebo"/>
-<xacro:include filename="transmission.xacro"/>
-<!-- dummy link -->
+<!-- <xacro:include filename="materials.xacro"/> -->
+<!-- <xacro:include filename="gazebo.gazebo"/> -->
+<!-- <xacro:include filename="transmission.xacro"/> -->
+<!-- dummy link (model root) -->
+<!-- see this post :
+	https://answers.ros.org/question/192817/error-msg-the-root-link_base-has-an-inertia-specified-in-the-urdf-but-kdl/
+	-->
 <link name="root_link">
 	<origin xyz="0 0 0" rpy="0 0 0"/>

Commit message: working on the manipulator

File: arm_urdf/urdf/arm.xacro (robot description, xacro)
@@ -1,6 +1,171 @@
 <?xml version="1.0" ?>
 <robot name="robot" xmlns:xacro="http://www.ros.org/wiki/xacro">
+<xacro:property name="arm_01_len" value="0.25" />
+<xacro:property name="arm_02_len" value="0.5" />
+<xacro:property name="arm_03_len" value="0.125" />
+<!-- base link of the manipulator -->
 <link name="arm_base_link">
-	<!-- ... -->
+	<origin
+		xyz="0 0 0"
+		rpy="0 0 0" />
+	<inertial>
+		<mass value="0.1"/>
+  		<origin xyz="0 0 0" rpy="0 0 0" />
+  		<inertia
+			ixx="0.0000416666667" iyy="0.0000416666667" izz="0.0000416666667"
+			iyz="0" ixy="0" ixz="0" />
+	</inertial>
+  	<collision>
+		<origin xyz="0 0 0" rpy="0 0 0"/>
+		<geometry>
+			<box size="0.1 0.1 0.1"/>
+		</geometry>
+  	</collision>
+  	<visual>
+		<origin xyz="0 0 0" rpy="0 0 0"/>
+		<geometry>
+			<box size="0.1 0.1 0.1"/>
+		</geometry>
+		<material name="red" />
+  	</visual>
 </link>
+<!-- base link of the manipulator -->
+<!-- first link of the manipulator -->
+<joint name="arm_joint_01" type="revolute">
+	<parent link="arm_base_link"/>
+	<child link="arm_link_01"/>
+	<origin rpy="0 0 0" xyz="0 0 ${arm_01_len/2}"/>
+	<axis xyz="0 0 1"/>
+	<limit effort="1000.0" lower="-3.14" upper="3.14" velocity="0.2"/>
+</joint>
+<link name="arm_link_01">
+	<origin
+		xyz="0 0 0"
+		rpy="0 0 0" />
+	<inertial>
+		<mass value="0.025"/>
+		<origin xyz="0 0 0" rpy="0 0 0" />
+		<inertia ixx="0.000010279" ixy="0" ixz="0" iyy="0.000010279" iyz="0" izz="0.000007225"/>
+	</inertial>
+	<collision>
+		<origin xyz="0 0 0" rpy="0 0 0"/>
+		<geometry>
+			<cylinder radius="0.04" length="${arm_01_len}"/>
+		</geometry>
+	</collision>
+	<visual>
+		<origin xyz="0 0 0" rpy="0 0 0"/>
+		<geometry>
+			<cylinder radius="0.04" length="${arm_01_len}"/>
+		</geometry>
+		<material name="red" />
+	</visual>
+</link>
+<!-- first link of the manipulator -->
+<!-- second link of the manipulator -->
+<joint name="arm_joint_02" type="revolute">
+	<parent link="arm_link_01"/>
+	<child link="arm_link_02"/>
+	<origin rpy="0 0 0" xyz="0 0 ${arm_02_len/2}"/>
+	<axis xyz="1 0 0"/>
+	<limit effort="1000.0" lower="-1.8" upper="1.8" velocity="0.2"/>
+</joint>
+<link name="arm_link_02">
+	<origin
+		xyz="0 0 0"
+		rpy="0 0 0" />
+	<inertial>
+		<mass value="0.025"/>
+		<origin xyz="0 0 0" rpy="0 0 0" />
+		<inertia
+			ixx="0.000010279" iyy="0.000010279" izz="0.000007225"
+			ixy="0" ixz="0" iyz="0"/>
+	</inertial>
+	<collision>
+		<origin xyz="0 0 ${arm_02_len/2}" rpy="0 0 0"/>
+		<geometry>
+			<cylinder radius="0.04" length="${arm_02_len}"/>
+		</geometry>
+	</collision>
+	<visual>
+		<origin xyz="0 0 ${arm_02_len/2}" rpy="0 0 0"/>
+		<geometry>
+			<cylinder radius="0.04" length="${arm_02_len}"/>
+		</geometry>
+		<material name="red" />
+	</visual>
+</link>
+<!-- second link of the manipulator -->
+<!-- third link of the manipulator -->
+<!--
+<joint name="arm_joint_03" type="revolute">
+	<parent link="arm_link_02"/>
+	<child link="arm_link_03"/>
+	<origin rpy="0 0 0" xyz="0 0 ${arm_03_len/2}"/>
+	<axis xyz="1 0 0"/>
+	<limit effort="1000.0" lower="-1.8" upper="1.8" velocity="0.2"/>
+</joint>
+<link name="arm_link_03">
+	<origin
+		xyz="0 0 0"
+		rpy="0 0 0" />
+	<inertial>
+		<mass value="0.025"/>
+		<origin xyz="0 0 0" rpy="0 0 0" />
+		<inertia
+			ixx="0.000010279" iyy="0.000010279" izz="0.000007225"
+			ixy="0" ixz="0" iyz="0"/>
+	</inertial>
+	<collision>
+		<origin xyz="0 0 0" rpy="0 0 0"/>
+		<geometry>
+			<cylinder radius="0.04" length="${arm_03_len}"/>
+		</geometry>
+	</collision>
+	<visual>
+		<origin xyz="0 0 0" rpy="0 0 0"/>
+		<geometry>
+			<cylinder radius="0.04" length="${arm_03_len}"/>
+		</geometry>
+		<material name="red" />
+	</visual>
+</link>
+-->
+<!-- third link of the manipulator -->
+<!-- last link of the manipulator -->
+<!--
+<joint name="arm_joint_04" type="revolute">
+	<parent link="arm_link_02"/>
+	<child link="arm_link_03"/>
+	<origin rpy="0 0 0" xyz="0 0 ${arm_04_len/2}"/>
+	<axis xyz="1 0 0"/>
+	<limit effort="1000.0" lower="-1.8" upper="1.8" velocity="0.2"/>
+</joint>
+<link name="arm_link_04">
+	<origin
+		xyz="0 0 0"
+		rpy="0 0 0" />
+	<inertial>
+		<mass value="0.025"/>
+		<origin xyz="0 0 0" rpy="0 0 0" />
+		<inertia
+			ixx="0.000010279" iyy="0.000010279" izz="0.000007225"
+			ixy="0" ixz="0" iyz="0"/>
+	</inertial>
+	<collision>
+		<origin xyz="0 0 0" rpy="0 0 0"/>
+		<geometry>
+			<cylinder radius="0.04" length="${arm_04_len}"/>
+		</geometry>
+	</collision>
+	<visual>
+		<origin xyz="0 0 0" rpy="0 0 0"/>
+		<geometry>
+			<cylinder radius="0.04" length="${arm_04_len}"/>
+		</geometry>
+		<material name="red" />
+	</visual>
+</link>
+-->
+<!-- last link of the manipulator -->
 </robot>

File: arm_urdf/urdf/main.xacro (robot description, xacro)
@@ -26,5 +26,5 @@
 	<parent link="base_link"/>
 	<child  link="arm_base_link"/>
-	<origin xyz="0 0 0" rpy="0 0 0"/>
+	<origin xyz="0 0 0.07" rpy="0 0 0"/>
 </joint>
 </robot>

Commit message: end of the work on the manipulator

File: arm_urdf/urdf/arm.xacro (robot description, xacro)
@@ -4,4 +4,6 @@
 <xacro:property name="arm_02_len" value="0.5" />
 <xacro:property name="arm_03_len" value="0.125" />
+<xacro:property name="arm_04_len" value="0.25" />
+<xacro:property name="offset" value="0" />
 <!-- base link of the manipulator -->
 <link name="arm_base_link">
@@ -35,7 +37,7 @@
 	<parent link="arm_base_link"/>
 	<child link="arm_link_01"/>
-	<origin rpy="0 0 0" xyz="0 0 ${arm_01_len/2}"/>
+	<origin rpy="0 0 0" xyz="0 0 ${0.05 + offset}"/>
 	<axis xyz="0 0 1"/>
-	<limit effort="1000.0" lower="-3.14" upper="3.14" velocity="0.2"/>
+	<limit effort="1000.0" lower="-3.12" upper="3.139" velocity="5"/>
 </joint>
 <link name="arm_link_01">
@@ -45,9 +47,9 @@
 	<inertial>
 		<mass value="0.025"/>
-		<origin xyz="0 0 0" rpy="0 0 0" />
+		<origin xyz="0 0 ${arm_01_len/2}" rpy="0 0 0" />
 		<inertia ixx="0.000010279" ixy="0" ixz="0" iyy="0.000010279" iyz="0" izz="0.000007225"/>
 	</inertial>
 	<collision>
-		<origin xyz="0 0 0" rpy="0 0 0"/>
+		<origin xyz="0 0 ${arm_01_len/2}" rpy="0 0 0"/>
 		<geometry>
 			<cylinder radius="0.04" length="${arm_01_len}"/>
@@ -55,5 +57,5 @@
 	</collision>
 	<visual>
-		<origin xyz="0 0 0" rpy="0 0 0"/>
+		<origin xyz="0 0 ${arm_01_len/2}" rpy="0 0 0"/>
 		<geometry>
 			<cylinder radius="0.04" length="${arm_01_len}"/>
@@ -67,7 +69,7 @@
 	<parent link="arm_link_01"/>
 	<child link="arm_link_02"/>
-	<origin rpy="0 0 0" xyz="0 0 ${arm_02_len/2}"/>
-	<axis xyz="1 0 0"/>
-	<limit effort="1000.0" lower="-1.8" upper="1.8" velocity="0.2"/>
+	<origin rpy="0 0 0" xyz="0 0 ${arm_01_len + offset}"/>
+	<axis xyz="0 1 0"/>
+	<limit effort="1000.0" lower="-1.8" upper="1.8" velocity="5"/>
 </joint>
 <link name="arm_link_02">
@@ -77,5 +79,5 @@
 	<inertial>
 		<mass value="0.025"/>
-		<origin xyz="0 0 0" rpy="0 0 0" />
+		<origin xyz="0 0 ${arm_02_len/2}" rpy="0 0 0" />
 		<inertia
 			ixx="0.000010279" iyy="0.000010279" izz="0.000007225"
@@ -98,11 +100,10 @@
 <!-- second link of the manipulator -->
 <!-- third link of the manipulator -->
-<!--
 <joint name="arm_joint_03" type="revolute">
 	<parent link="arm_link_02"/>
 	<child link="arm_link_03"/>
-	<origin rpy="0 0 0" xyz="0 0 ${arm_03_len/2}"/>
-	<axis xyz="1 0 0"/>
-	<limit effort="1000.0" lower="-1.8" upper="1.8" velocity="0.2"/>
+	<origin rpy="0 0 0" xyz="0 0 ${arm_02_len + offset}"/>
+	<axis xyz="0 1 0"/>
+	<limit effort="1000.0" lower="-1.8" upper="1.8" velocity="5"/>
 </joint>
 <link name="arm_link_03">
@@ -112,5 +113,5 @@
 	<inertial>
 		<mass value="0.025"/>
-		<origin xyz="0 0 0" rpy="0 0 0" />
+		<origin xyz="0 0 ${arm_03_len/2}" rpy="0 0 0" />
 		<inertia
 			ixx="0.000010279" iyy="0.000010279" izz="0.000007225"
@@ -118,5 +119,5 @@
 	</inertial>
 	<collision>
-		<origin xyz="0 0 0" rpy="0 0 0"/>
+		<origin xyz="0 0 ${arm_03_len/2}" rpy="0 0 0"/>
 		<geometry>
 			<cylinder radius="0.04" length="${arm_03_len}"/>
@@ -124,5 +125,5 @@
 	</collision>
 	<visual>
-		<origin xyz="0 0 0" rpy="0 0 0"/>
+		<origin xyz="0 0 ${arm_03_len/2}" rpy="0 0 0"/>
 		<geometry>
 			<cylinder radius="0.04" length="${arm_03_len}"/>
@@ -131,14 +132,12 @@
 	</visual>
 </link>
--->
 <!-- third link of the manipulator -->
-<!-- last link of the manipulator -->
-<!--
+<!-- last link of the manipulator, base gripper -->
 <joint name="arm_joint_04" type="revolute">
-	<parent link="arm_link_02"/>
-	<child link="arm_link_03"/>
-	<origin rpy="0 0 0" xyz="0 0 ${arm_04_len/2}"/>
-	<axis xyz="1 0 0"/>
-	<limit effort="1000.0" lower="-1.8" upper="1.8" velocity="0.2"/>
+	<parent link="arm_link_03"/>
+	<child link="arm_link_04"/>
+	<origin rpy="0 0 0" xyz="0 0 ${arm_03_len + offset}"/>
+	<axis xyz="0 1 0"/>
+	<limit effort="1000.0" lower="-1.8" upper="1.8" velocity="5"/>
 </joint>
 <link name="arm_link_04">
@@ -148,5 +147,5 @@
 	<inertial>
 		<mass value="0.025"/>
-		<origin xyz="0 0 0" rpy="0 0 0" />
+		<origin xyz="0 0 0.04" rpy="0 0 0" />
 		<inertia
 			ixx="0.000010279" iyy="0.000010279" izz="0.000007225"
@@ -154,13 +153,13 @@
 	</inertial>
 	<collision>
-		<origin xyz="0 0 0" rpy="0 0 0"/>
-		<geometry>
-			<cylinder radius="0.04" length="${arm_04_len}"/>
-		</geometry>
-	</collision>
-	<visual>
-		<origin xyz="0 0 0" rpy="0 0 0"/>
-		<geometry>
-			<cylinder radius="0.04" length="${arm_04_len}"/>
+		<origin xyz="0 0 0.04" rpy="0 0 0"/>
+		<geometry>
+			<box size="0.034 0.2 0.08"/>
+		</geometry>
+	</collision>
+	<visual>
+		<origin xyz="0 0 0.04" rpy="0 0 0"/>
+		<geometry>
+			<box size="0.034 0.2 0.08"/>
 		</geometry>
 		<material name="red" />
@@ -168,4 +167,68 @@
 </link>
 -->
-<!-- last link of the manipulator -->
+<!-- last link of the manipulator, base gripper -->
+<!-- right gripper -->
+<joint name="right_grip_joint" type="prismatic">
+	<parent link="arm_link_04"/>
+	<child link="right_grip_link"/>
+	<origin rpy="0 0 0" xyz="${0.015 + 0.03} 0.05 0.04"/>
+	<axis xyz="0 1 0"/>
+	<limit effort="1000.0" lower="-0.04" upper="0.035" velocity="6.5"/>
+</joint>
+<link name="right_grip_link">
+	<origin
+		xyz="0 0 0"
+		rpy="0 0 0" />
+	<inertial>
+		<mass value="0.01"/>
+		<origin xyz="0 0 0" rpy="0 0 0" />
+		<inertia ixx="0.000010279" ixy="0" ixz="0" iyy="0.000010279" iyz="0" izz="0.000007225"/>
+	</inertial>
+	<collision>
+		<origin rpy="0 0 0" xyz="0 0 0"/>
+		<geometry>
+			<box size="0.06 0.02 0.08"/>
+		</geometry>
+	</collision>
+  	<visual>
+		<origin rpy="0 0 0" xyz="0 0 0"/>
+		<geometry>
+			<box size="0.06 0.02 0.08"/>
+		</geometry>
+		<material name="white" />
+  	</visual>
+</link>
+<!-- right gripper -->
+<!-- left gripper -->
+<joint name="left_grip_joint" type="prismatic">
+	<parent link="arm_link_04"/>
+	<child link="left_grip_link"/>
+	<origin rpy="0 0 0" xyz="${0.015 + 0.03} -0.05 0.04"/>
+	<axis xyz="0 1 0"/>
+	<limit effort="1000.0" upper="0.04" lower="-0.035" velocity="6.5"/>
+</joint>
+<link name="left_grip_link">
+	<origin
+		xyz="0 0 0"
+		rpy="0 0 0" />
+  	<inertial>
+		<mass value="0.01"/>
+		<origin xyz="0 0 0" rpy="0 0 0" />
+		<inertia ixx="0.000010279" ixy="0" ixz="0" iyy="0.000010279" iyz="0" izz="0.000007225"/>
+  	</inertial>
+  	<collision>
+		<origin rpy="0 0 0" xyz="0 0 0"/>
+		<geometry>
+			<box size="0.06 0.02 0.08"/>
+		</geometry>
+  	</collision>
+  	<visual>
+		<origin rpy="0 0 0" xyz="0 0 0"/>
+		<geometry>
+			<box size="0.06 0.02 0.08"/>
+		</geometry>
+		<material name="white" />
+  	</visual>
+</link>
+<!-- left gripper -->
 </robot>

File: arm_urdf/urdf/chassis.xacro (robot description, xacro)
@@ -9,5 +9,5 @@
 		<origin
 			rpy="0 0 0"
-			xyz="0 0 0.1"/>
+			xyz="0 0 0"/>
 		<inertia
 			ixx="0.0395416666667" iyy="0.106208333333" izz="0.106208333333"
@@ -59,4 +59,9 @@
 <!-- chassis and front caster wheel -->
 <!-- place for laser sensors -->
+<joint name="joint_laser" type="fixed">
+	<parent link="base_link"/>
+	<child link="laser"/>
+	<origin xyz="0.15 0 0.05" rpy="0 0 0"/>
+</joint>
 <link name="laser">
 	<inertial>
@@ -79,9 +84,4 @@
 	</collision>
 </link>
-<joint name="joint_laser" type="fixed">
-	<parent link="base_link"/>
-	<child link="laser"/>
-	<origin xyz="0.15 0 0.05" rpy="0 0 0"/>
-</joint>
 <!-- place for laser sensors -->
 <!-- Wheels -->

File: arm_urdf/urdf/main.xacro (robot description, xacro)
@@ -5,6 +5,6 @@
 <xacro:include filename="params.xacro"/>
 <xacro:include filename="materials.xacro"/>
-<!-- <xacro:include filename="gazebo.gazebo"/> -->
-<!-- <xacro:include filename="transmission.xacro"/> -->
+<xacro:include filename="gazebo.gazebo"/>
+<xacro:include filename="transmission.xacro"/>
 <!-- dummy link (model root) -->
 <!-- see this post :
@@ -26,5 +26,6 @@
 	<parent link="base_link"/>
 	<child  link="arm_base_link"/>
-	<origin xyz="0 0 0.07" rpy="0 0 0"/>
+	<!-- origin : 0.5*(chassis height) + 0.5*(arm base link height) -->
+	<origin xyz="0 0 0.085" rpy="0 0 0"/>
 </joint>
 </robot>

Commit message: controllers added to the model; setting Gazebo

File: arm_urdf/urdf/arm.xacro (robot description, xacro)
@@ -1,8 +1,12 @@
 <?xml version="1.0" ?>
 <robot name="robot" xmlns:xacro="http://www.ros.org/wiki/xacro">
-<xacro:property name="arm_01_len" value="0.25" />
-<xacro:property name="arm_02_len" value="0.5" />
-<xacro:property name="arm_03_len" value="0.125" />
+<xacro:property name="arm_01_len" value="0.2" />
+<xacro:property name="arm_01_mass" value="0.025" />
+<xacro:property name="arm_02_len" value="0.2" />
+<xacro:property name="arm_02_mass" value="0.025" />
+<xacro:property name="arm_03_len" value="0.2" />
+<xacro:property name="arm_03_mass" value="0.025" />
 <xacro:property name="arm_04_len" value="0.25" />
+<xacro:property name="arm_04_mass" value="0.025" />
 <xacro:property name="offset" value="0" />
 <!-- base link of the manipulator -->
@@ -46,7 +50,7 @@
 		rpy="0 0 0" />
 	<inertial>
-		<mass value="0.025"/>
 		<origin xyz="0 0 ${arm_01_len/2}" rpy="0 0 0" />
-		<inertia ixx="0.000010279" ixy="0" ixz="0" iyy="0.000010279" iyz="0" izz="0.000007225"/>
+		<mass value="${arm_01_mass}"/>
+		<xacro:cylinder_inertia mass="${arm_01_mass}" r="0.04" l="${arm_01_len}" />
 	</inertial>
 	<collision>
@@ -78,9 +82,7 @@
 		rpy="0 0 0" />
 	<inertial>
-		<mass value="0.025"/>
 		<origin xyz="0 0 ${arm_02_len/2}" rpy="0 0 0" />
-		<inertia
-			ixx="0.000010279" iyy="0.000010279" izz="0.000007225"
-			ixy="0" ixz="0" iyz="0"/>
+		<mass value="${arm_02_mass}"/>
+		<xacro:cylinder_inertia mass="${arm_02_mass}" r="0.04" l="${arm_02_len}" />
 	</inertial>
 	<collision>
@@ -112,9 +114,7 @@
 		rpy="0 0 0" />
 	<inertial>
-		<mass value="0.025"/>
 		<origin xyz="0 0 ${arm_03_len/2}" rpy="0 0 0" />
-		<inertia
-			ixx="0.000010279" iyy="0.000010279" izz="0.000007225"
-			ixy="0" ixz="0" iyz="0"/>
+		<mass value="${arm_03_mass}"/>
+		<xacro:cylinder_inertia mass="${arm_03_mass}" r="0.04" l="${arm_03_len}" />
 	</inertial>
 	<collision>
@@ -139,5 +139,5 @@
 	<origin rpy="0 0 0" xyz="0 0 ${arm_03_len + offset}"/>
 	<axis xyz="0 1 0"/>
-	<limit effort="1000.0" lower="-1.8" upper="1.8" velocity="5"/>
+	<limit effort="10000.0" lower="-1.8" upper="1.8" velocity="5"/>
 </joint>
 <link name="arm_link_04">
@@ -146,6 +146,6 @@
 		rpy="0 0 0" />
 	<inertial>
-		<mass value="0.025"/>
 		<origin xyz="0 0 0.04" rpy="0 0 0" />
+		<mass value="${arm_04_mass}"/>
 		<inertia
 			ixx="0.000010279" iyy="0.000010279" izz="0.000007225"

File: arm_urdf/urdf/macros.xacro (robot description, xacro)
@@ -6,4 +6,7 @@
 -->
 <!-- Inertia Matrix of the cilinder -->
+<!--
+<xacro:cylinder_inertia mass="" r="" l="" />
+-->
 <xacro:macro name="cylinder_inertia" params="mass r l">
 	<inertia
@@ -11,4 +14,5 @@
 		ixy = "0" ixz = "0" iyz = "0" />
 </xacro:macro>
+<!-- Inertia Matrix of the cilinder -->
 <!-- link of the wheel of the chassis (use this alongside with joint_wheel) -->
 <xacro:macro name="link_wheel" params="name">
@@ -44,4 +48,5 @@
 	</link>
 </xacro:macro>
+<!-- link of the wheel of the chassis (use this alongside with joint_wheel) -->
 <!-- joint of the wheel on the chassis -->
 <xacro:macro name="joint_wheel" params="name child parent xx yy zz">
@@ -59,3 +64,4 @@
 	</joint>
 </xacro:macro>
+<!-- joint of the wheel on the chassis -->
 </robot>

Commit message: arm_link_04 -> cluedo_link; rearranging urdf model script generator

File: arm_urdf/urdf/arm.xacro (robot description, xacro)
@@ -136,10 +136,10 @@
 <joint name="arm_joint_04" type="revolute">
 	<parent link="arm_link_03"/>
-	<child link="arm_link_04"/>
+	<child link="cluedo_link"/>
 	<origin rpy="0 0 0" xyz="0 0 ${arm_03_len + offset}"/>
 	<axis xyz="0 1 0"/>
 	<limit effort="10000.0" lower="-1.8" upper="1.8" velocity="5"/>
 </joint>
-<link name="arm_link_04">
+<link name="cluedo_link">
 	<origin
 		xyz="0 0 0"
@@ -170,5 +170,5 @@
 <!-- right gripper -->
 <joint name="right_grip_joint" type="prismatic">
-	<parent link="arm_link_04"/>
+	<parent link="cluedo_link"/>
 	<child link="right_grip_link"/>
 	<origin rpy="0 0 0" xyz="${0.015 + 0.03} 0.05 0.04"/>
@@ -202,5 +202,5 @@
 <!-- left gripper -->
 <joint name="left_grip_joint" type="prismatic">
-	<parent link="arm_link_04"/>
+	<parent link="cluedo_link"/>
 	<child link="left_grip_link"/>
 	<origin rpy="0 0 0" xyz="${0.015 + 0.03} -0.05 0.04"/>

Commit message: testing with move_base

File: arm_urdf/urdf/arm.xacro (robot description, xacro)
@@ -43,5 +43,5 @@
 	<origin rpy="0 0 0" xyz="0 0 ${0.05 + offset}"/>
 	<axis xyz="0 0 1"/>
-	<limit effort="1000.0" lower="-3.12" upper="3.139" velocity="5"/>
+	<limit effort="1000000.0" lower="-3.12" upper="3.139" velocity="5"/>
 </joint>
 <link name="arm_link_01">
@@ -75,5 +75,5 @@
 	<origin rpy="0 0 0" xyz="0 0 ${arm_01_len + offset}"/>
 	<axis xyz="0 1 0"/>
-	<limit effort="1000.0" lower="-1.8" upper="1.8" velocity="5"/>
+	<limit effort="1000000.0" lower="-1.8" upper="1.8" velocity="5"/>
 </joint>
 <link name="arm_link_02">
@@ -107,5 +107,5 @@
 	<origin rpy="0 0 0" xyz="0 0 ${arm_02_len + offset}"/>
 	<axis xyz="0 1 0"/>
-	<limit effort="1000.0" lower="-1.8" upper="1.8" velocity="5"/>
+	<limit effort="1000000.0" lower="-1.8" upper="1.8" velocity="5"/>
 </joint>
 <link name="arm_link_03">
@@ -139,5 +139,5 @@
 	<origin rpy="0 0 0" xyz="0 0 ${arm_03_len + offset}"/>
 	<axis xyz="0 1 0"/>
-	<limit effort="10000.0" lower="-1.8" upper="1.8" velocity="5"/>
+	<limit effort="10000000.0" lower="-1.8" upper="1.8" velocity="5"/>
 </joint>
 <link name="cluedo_link">
@@ -174,5 +174,5 @@
 	<origin rpy="0 0 0" xyz="${0.015 + 0.03} 0.05 0.04"/>
 	<axis xyz="0 1 0"/>
-	<limit effort="1000.0" lower="-0.04" upper="0.035" velocity="6.5"/>
+	<limit effort="1000000.0" lower="-0.04" upper="0.035" velocity="6.5"/>
 </joint>
 <link name="right_grip_link">
@@ -206,5 +206,5 @@
 	<origin rpy="0 0 0" xyz="${0.015 + 0.03} -0.05 0.04"/>
 	<axis xyz="0 1 0"/>
-	<limit effort="1000.0" upper="0.04" lower="-0.035" velocity="6.5"/>
+	<limit effort="1000000.0" upper="0.04" lower="-0.035" velocity="6.5"/>
 </joint>
 <link name="left_grip_link">

File: arm_urdf/urdf/chassis.xacro (robot description, xacro)
@@ -86,4 +86,5 @@
 <!-- place for laser sensors -->
 <!-- Wheels -->
+<!--
 <xacro:link_wheel name="link_right_wheel" />
 <xacro:joint_wheel name="joint_right_wheel"
@@ -92,4 +93,61 @@
 <xacro:joint_wheel name="joint_left_wheel"
 	child="link_left_wheel" parent="base_link" xx="-0.05" yy="-0.15" zz="0"  />
+-->
+<link name="link_right_wheel">
+	<inertial>
+		<mass value="0.2"/>
+		<origin rpy="0 1.5707 1.5707" xyz="0 0 0"/>
+		<inertia ixx="0.000526666666667" ixy="0" ixz="0" iyy="0.000526666666667" iyz="0" izz="0.001"/>
+	</inertial>
+	<collision name="link_right_wheel_collision">
+		<origin rpy="0 1.5707 1.5707" xyz="0 0 0"/>
+		<geometry>
+			<cylinder length="0.04" radius="0.1"/>
+		</geometry>
+	</collision>
+	<visual name="link_right_wheel_visual">
+		<origin rpy="0 1.5707 1.5707" xyz="0 0 0"/>
+		<geometry>
+			<cylinder length="0.04" radius="0.1"/>
+		</geometry>
+		<material name="red"/>
+	</visual>
+</link>
+<link name="link_left_wheel">
+	<inertial>
+		<mass value="0.2"/>
+		<origin rpy="0 1.5707 1.5707" xyz="0 0 0"/>
+		<inertia ixx="0.000526666666667" ixy="0" ixz="0" iyy="0.000526666666667" iyz="0" izz="0.001"/>
+	</inertial>
+	<collision name="link_left_wheel_collision">
+		<origin rpy="0 1.5707 1.5707" xyz="0 0 0"/>
+		<geometry>
+			<cylinder length="0.04" radius="0.1"/>
+		</geometry>
+	</collision>
+	<visual name="link_left_wheel_visual">
+		<origin rpy="0 1.5707 1.5707" xyz="0 0 0"/>
+		<geometry>
+			<cylinder length="0.04" radius="0.1"/>
+		</geometry>
+		<material name="red"/>
+	</visual>
+</link>
+<joint name="joint_right_wheel" type="continuous">
+	<origin rpy="0 0 0" xyz="-0.05 0.15 0"/>
+	<child link="link_right_wheel"/>
+	<parent link="base_link"/>
+	<axis rpy="0 0 0" xyz="0 1 0"/>
+	<limit effort="10000" velocity="1000"/>
+	<joint_properties damping="1.0" friction="1.0"/>
+</joint>
+<joint name="joint_left_wheel" type="continuous">
+	<origin rpy="0 0 0" xyz="-0.05 -0.15 0"/>
+	<child link="link_left_wheel"/>
+	<parent link="base_link"/>
+	<axis rpy="0 0 0" xyz="0 1 0"/>
+	<limit effort="10000" velocity="1000"/>
+	<joint_properties damping="1.0" friction="1.0"/>
+</joint>
 <!-- Wheels -->
 </robot>

File: arm_urdf/urdf/main.xacro (robot description, xacro)
@@ -10,9 +10,11 @@
 	https://answers.ros.org/question/192817/error-msg-the-root-link_base-has-an-inertia-specified-in-the-urdf-but-kdl/
 	-->
+<!--
 <link name="root_link">
 	<origin xyz="0 0 0" rpy="0 0 0"/>
-</link>
+</link>-->
 <!-- robot chassis -->
 <xacro:include filename="chassis.xacro"></xacro:include>
+<!--
 <joint name="root_joint" type="fixed">
 	<parent link="root_link"/>
@@ -20,4 +22,5 @@
 	<origin xyz="0 0 0" rpy="0 0 0"/>
 </joint>
+-->
 <!-- robot manipulator -->
 <xacro:include filename="arm.xacro"></xacro:include>

File: arm_urdf/urdf/model/model.urdf (robot description, URDF)
Before this commit: robot robot, 12 links, 11 joints
Links:
- removed link root_link
Joints:
- removed joint root_joint
